File: Overview & Details/Week_3/Week_3_Activity/Activity_3/activity3/activity3.sch (KiCad schematic (older format))
At the start: 2 parts, among them J1 62684-502100ALF, U3 DISP_TFT_2.8IN_240x320_50PIN

Commit message: linked FFC and STMPE811 symbols with their respective footprints
Parts:
- J1: footprint Display_Board:62684-502100ALF -> activity3:62684-502100ALF
Changed lines of the file:
@@
 F 0 "J1" H 6300 1570 60  0000 L CNN
 F 1 "62684-502100ALF" H 6050 1630 60  0000 L CNN
-F 2 "Display_Board:62684-502100ALF" H 6400 -1040 60  0001 C CNN
+F 2 "activity3:62684-502100ALF" H 6400 -1040 60  0001 C CNN
 F 3 "" H 6000 1420 60  0000 C CNN
 	1    6000 1420
